File: KICAD Files/NLIME_Slime.kicad_sch (KiCad schematic)
At the start: 21 parts, among them SW2 SWO, SW3 SW_Push, U2 QMC6309, U3 ICM-45686, X1 32.768MHz

Commit message: Add files via upload
Parts:
- C4: LCSC C12530 -> C23630
Connections:
- net -BATT_SWT is gone; now on net GND: SW1.2 (B), U1.1 (B-)
Changed lines of the file:
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@@
 	)
 	(no_connect
-		(at 168.91 50.8)
+		(at 168.91 63.5)
 	)
 	(no_connect
-		(at 168.91 63.5)
+		(at 168.91 50.8)
 	)
 	(no_connect
@@
 	(wire
 		(pts
-			(xy 138.43 48.26) (xy 132.08 48.26)
-		)
-		(stroke
-			(width 0)
-			(type default)
-		)
-	)
-	(wire
-		(pts
 			(xy 132.08 68.58) (xy 138.43 68.58)
 		)
@@
 	(wire
 		(pts
+			(xy 120.65 48.26) (xy 138.43 48.26)
+		)
+		(stroke
+			(width 0)
+			(type default)
+		)
+	)
+	(wire
+		(pts
 			(xy 132.08 53.34) (xy 138.43 53.34)
 		)
@@
 	(wire
 		(pts
-			(xy 132.08 48.26) (xy 132.08 43.18)
+			(xy 67.31 86.36) (xy 69.85 86.36)
 		)
 		(stroke
@@
 	(wire
 		(pts
-			(xy 67.31 86.36) (xy 69.85 86.36)
+			(xy 153.67 86.36) (xy 156.21 86.36)
 		)
 		(stroke
@@
 	(wire
 		(pts
-			(xy 153.67 86.36) (xy 156.21 86.36)
+			(xy 151.13 83.82) (xy 151.13 86.36)
 		)
 		(stroke
@@
 	(wire
 		(pts
-			(xy 151.13 83.82) (xy 151.13 86.36)
+			(xy 24.13 35.56) (xy 24.13 36.83)
 		)
 		(stroke
@@
 			)
 		)
-		(property "LCSC" "C12530"
+		(property "LCSC" "C23630"
 			(at 93.98 44.45 90)
 			(effects
@@
 	)
 	(symbol
-		(lib_id "power:-BATT")
-		(at 132.08 43.18 0)
+		(lib_id "NLIME_Slimes:Battery_302025")
+		(at 53.34 177.8 0)
 		(unit 1)
-		(exclude_from_sim no)
-		(in_bom yes)
+		(exclude_from_sim yes)
+		(in_bom no)
 		(on_board yes)
-		(dnp no)
+		(dnp yes)
 		(fields_autoplaced yes)
-		(property "Reference" "#PWR09"
-			(at 132.08 46.99 0)
+		(property "Reference" "BT2"
+			(at 57.15 174.6884 0)
 			(effects
 				(font
 					(size 1.27 1.27)
 				)
-				(hide yes)
+				(justify left)
 			)
 		)
-		(property "Value" "-BATT_SWT"
-			(at 132.08 38.1 0)
+		(property "Value" "Battery_302025"
+			(at 57.15 177.2284 0)
 			(effects
 				(font
 					(size 1.27 1.27)
 				)
+				(justify left)
 			)
 		)
-		(property "Footprint" ""
-			(at 132.08 43.18 0)
+		(property "Footprint" "NLIME_Slimes:302025 Bat Rep"
+			(at 53.34 176.276 90)
 			(effects
 				(font
@@
 			)
 		)
-		(property "Datasheet" ""
-			(at 132.08 43.18 0)
+		(property "Datasheet" "~"
+			(at 53.34 176.276 90)
 			(effects
 				(font
@@
 			)
 		)
-		(property "Description" "Power symbol creates a global label with name \"-BATT\""
-			(at 132.08 43.18 0)
+		(property "Description" "Single-cell battery"
+			(at 53.34 177.8 0)
 			(effects
 				(font
@@
 			)
 		)
+		(pin "2"
+		)
 		(pin "1"
 		)
 		(instances
-			(project "SlimeButterfly"
+			(project ""
 				(path "/95168c8f-ea80-49b0-8f73-f32d7ec2a49f"
-					(reference "#PWR09")
+					(reference "BT2")
 					(unit 1)
 				)
@@
 	)
 	(symbol
-		(lib_id "NLIME_Slimes:Battery_302025")
-		(at 53.34 177.8 0)
+		(lib_id "power:GND")
+		(at 24.13 36.83 0)
 		(unit 1)
-		(exclude_from_sim yes)
-		(in_bom no)
+		(exclude_from_sim no)
+		(in_bom yes)
 		(on_board yes)
-		(dnp yes)
+		(dnp no)
 		(fields_autoplaced yes)
-		(property "Reference" "BT2"
-			(at 57.15 174.6884 0)
+		(property "Reference" "#PWR025"
+			(at 24.13 43.18 0)
 			(effects
 				(font
 					(size 1.27 1.27)
 				)
-				(justify left)
+				(hide yes)
 			)
 		)
-		(property "Value" "Battery_302025"
-			(at 57.15 177.2284 0)
+		(property "Value" "GND"
+			(at 24.13 41.91 0)
 			(effects
 				(font
 					(size 1.27 1.27)
 				)
-				(justify left)
 			)
 		)
-		(property "Footprint" "NLIME_Slimes:302025 Bat Rep"
-			(at 53.34 176.276 90)
+		(property "Footprint" ""
+			(at 24.13 36.83 0)
 			(effects
 				(font
@@
 			)
 		)
-		(property "Datasheet" "~"
-			(at 53.34 176.276 90)
+		(property "Datasheet" ""
+			(at 24.13 36.83 0)
 			(effects
 				(font
@@
 			)
 		)
-		(property "Description" "Single-cell battery"
-			(at 53.34 177.8 0)
+		(property "Description" "Power symbol creates a global label with name \"GND\" , ground"
+			(at 24.13 36.83 0)
 			(effects
 				(font
@@
 			)
 		)
-		(pin "2"
-		)
 		(pin "1"
 		)
 		(instances
-			(project ""
+			(project "NLIME_Slime"
 				(path "/95168c8f-ea80-49b0-8f73-f32d7ec2a49f"
-					(reference "BT2")
+					(reference "#PWR025")
 					(unit 1)
 				)
@@
 	)
 	(symbol
-		(lib_id "power:-BATT")
-		(at 24.13 35.56 0)
-		(unit 1)
-		(exclude_from_sim no)
-		(in_bom yes)
-		(on_board yes)
-		(dnp no)
-		(fields_autoplaced yes)
-		(property "Reference" "#PWR07"
-			(at 24.13 39.37 0)
-			(effects
-				(font
-					(size 1.27 1.27)
-				)
-				(hide yes)
-			)
-		)
-		(property "Value" "-BATT_SWT"
-			(at 24.13 30.48 0)
-			(effects
-				(font
-					(size 1.27 1.27)
-				)
-			)
-		)
-		(property "Footprint" ""
-			(at 24.13 35.56 0)
-			(effects
-				(font
-					(size 1.27 1.27)
-				)
-				(hide yes)
-			)
-		)
-		(property "Datasheet" ""
-			(at 24.13 35.56 0)
-			(effects
-				(font
-					(size 1.27 1.27)
-				)
-				(hide yes)
-			)
-		)
-		(property "Description" "Power symbol creates a global label with name \"-BATT\""
-			(at 24.13 35.56 0)
-			(effects
-				(font
-					(size 1.27 1.27)
-				)
-				(hide yes)
-			)
-		)
-		(pin "1"
-		)
-		(instances
-			(project "SlimeButterfly"
-				(path "/95168c8f-ea80-49b0-8f73-f32d7ec2a49f"
-					(reference "#PWR07")
-					(unit 1)
-				)
-			)
-		)
-	)
-	(symbol
 		(lib_id "power:GND")
 		(at 223.52 49.53 0)
@@
 					(unit 1)
 				)
+			)
+		)
+	)
+	(symbol
+		(lib_id "power:GND")
+		(at 120.65 48.26 0)
+		(unit 1)
+		(exclude_from_sim no)
+		(in_bom yes)
+		(on_board yes)
+		(dnp no)
+		(fields_autoplaced yes)
+		(property "Reference" "#PWR02"
+			(at 120.65 54.61 0)
+			(effects
+				(font
+					(size 1.27 1.27)
+				)
+				(hide yes)
+			)
+		)
+		(property "Value" "GND"
+			(at 120.65 53.34 0)
+			(effects
+				(font
+					(size 1.27 1.27)
+				)
+			)
+		)
+		(property "Footprint" ""
+			(at 120.65 48.26 0)
+			(effects
+				(font
+					(size 1.27 1.27)
+				)
+				(hide yes)
+			)
+		)
+		(property "Datasheet" ""
+			(at 120.65 48.26 0)
+			(effects
+				(font
+					(size 1.27 1.27)
+				)
+				(hide yes)
+			)
+		)
+		(property "Description" "Power symbol creates a global label with name \"GND\" , ground"
+			(at 120.65 48.26 0)
+			(effects
+				(font
+					(size 1.27 1.27)
+				)
+				(hide yes)
+			)
+		)
+		(pin "1"
+		)
+		(instances
+			(project "NLIME_Slime"
+				(path "/95168c8f-ea80-49b0-8f73-f32d7ec2a49f"
+					(reference "#PWR02")
+					(unit 1)
+				)
