File: KICAD Files/NLIME_Slime.kicad_pcb (KiCad board)
At the start: 2 copper layers, 32.5 x 34.5 mm, 28 parts, among them SW2 SWO, SW3 SW_Push, U2 QMC6309, U3 ICM-45686, X1 32.768MHz

Commit message: Add files via upload
Parts:
- moved G*** 2.25 mm to (21.6, 21.2)
- moved BT1 0.43 mm to (21.8, 17.5)
Routing:
- net +BATT: track 12.6 -> 10.1 mm
- net GND: vias 9 -> 11

Commit message: Add files via upload
Parts:
- moved REF** 0.43 mm to (16.9, 16.5)
Connections:
- SW1 pad 2: -BATT_SWT -> GND
- U1 pad 1: -BATT_SWT -> GND
Routing:
- net -BATT_SWT: track 26.1 -> 0.00 mm
- net GND: track 5.49 -> 17.4 mm
- net +3V3: track 69.7 -> 68.7 mm, vias 6 -> 8

Commit message: Add files via upload
Parts:
- moved REF** 0.38 mm to (16.9, 46.8)
Routing:
- added copper zone on In1.Cu, net GND
- added copper zone on In2.Cu, net GND
Other:
- outline, holes or cut-outs redrawn
- copper layers 2 -> 4
